File: pcb/bakeneko-65-pcb.kicad_pcb (KiCad board)
At the start: 2 copper layers, 303.8 x 94.2 mm, 161 parts, among them J1 JST SH 4-pin, J2 AVR-ISP-6, SW1 Reset, U1 SRV05-4, U2 ATmega32U4-AU, Y1 16MHz

Commit message: Original Commit
Changed to MU compared to 32u4 AU, changed to hotswap sockets
Parts:
- MX1, MX10, MX11, MX12, MX13, MX14, MX15, MX16, MX19, MX2, MX20, MX21, MX22, MX23, MX24, MX25, MX26, MX27, MX28, MX29, MX3, MX30, MX32, MX35, MX36, MX37, MX38, MX39, MX4, MX40, MX41, MX42, MX43, MX44, MX45, MX47, MX49, MX5, MX50, MX51, MX52, MX53, MX54, MX55, MX56, MX57, MX58, MX6, MX60, MX61, MX63, MX68, MX69, MX7, MX70, MX8, MX9: footprint MX_Only:MXOnly-1U-NoLED -> MX_HS:MXOnly-1U-Hotswap-NoLED; moved to B.Cu
- MX17: footprint MX_Only:MXOnly-2U-NoLED -> MX_HS:MXOnly-2U-Hotswap-NoLED; moved to B.Cu
- MX18, MX31, MX62, MX64, MX67: footprint MX_Only:MXOnly-1.5U-NoLED -> MX_HS:MXOnly-1.5U-Hotswap-NoLED; moved to B.Cu
- MX33, MX66, MX71, MX72, MX73, MX75: footprint MX_Only:MXOnly-1.25U-NoLED -> MX_HS:MXOnly-1.25U-Hotswap-NoLED; moved to B.Cu
- MX34, MX59: footprint MX_Only:MXOnly-1.75U-NoLED -> MX_HS:MXOnly-1.75U-Hotswap-NoLED; moved to B.Cu
- MX46, MX48: footprint MX_Only:MXOnly-2.25U-NoLED -> MX_HS:MXOnly-2.25U-Hotswap-NoLED; moved to B.Cu
- MX65: footprint MX_Only:MXOnly-7U-ReversedStabilizers-NoLED -> MX_HS:MXOnly-7U-Hotswap-NoLED; moved to B.Cu
- MX74: footprint MX_Only:MXOnly-6.25U-ReversedStabilizers-NoLED -> MX_HS:MXOnly-6.25U-Hotswap-NoLED; moved to B.Cu
- U2: footprint Package_QFP:TQFP-44_10x10mm_P0.8mm -> Package_DFN_QFN:QFN-44-1EP_7x7mm_P0.5mm_EP5.2x5.2mm
- moved D1 14.8 mm to (2.38, 12.7)
- moved R4 13.5 mm to (24.9, 43.4)
- moved D15 6.19 mm to (284.8, 15.9)
- moved D66 5.96 mm to (260.2, 90.0)
- moved D67 5.91 mm to (272.1, 90.0)
- moved D16 5.72 mm to (288.0, 15.4)
- moved C2 5.27 mm to (22.1, 40.5)
- moved D68 4.20 mm to (284.0, 90.0)
- moved D32 3.59 mm to (26.2, 50.8)
- moved C3 2.93 mm to (31.7, 44.0), turned to 90 degrees
- moved D2 2.65 mm to (17.5, 9.80)
- moved D62 2.28 mm to (50.8, 84.1)
- moved C7 2.16 mm to (28.5, 29.6)
- moved C1 2.04 mm to (35.1, 34.2)
- moved D60 1.93 mm to (22.2, 84.1)
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Connections:
- U1 pad 3: Net-(U1-Pad3) -> unconnected-(U1-Pad3)
- U1 pad 4: Net-(U1-Pad4) -> unconnected-(U1-Pad4)
- U2 pad 41: Net-(U2-Pad41) -> unconnected-(U2-Pad41)
- U2 pad 42: Net-(U2-Pad42) -> unconnected-(U2-Pad42)
Routing:
- net ROW0: track 295.7 -> 327.4 mm
- net ROW4: track 346.6 -> 376.8 mm
- net GND: track 184.5 -> 156.6 mm
- net COL11: track 293.6 -> 317.0 mm
- net COL1: track 113.8 -> 136.0 mm
- net COL2: track 143.6 -> 164.7 mm
- net Net-(D63-Pad2): track 18.7 -> 35.8 mm
- net COL0: track 99.8 -> 116.7 mm
- net ROW2: track 301.5 -> 286.7 mm
- net Net-(D65-Pad2): track 9.20 -> 22.1 mm
- net Net-(R4-Pad2): track 14.6 -> 1.81 mm
- net Net-(D61-Pad2): track 9.20 -> 20.6 mm
- net Net-(D14-Pad2): track 6.82 -> 18.0 mm
- net Net-(D62-Pad2): track 9.20 -> 19.4 mm
- net Net-(D60-Pad2): track 15.2 -> 25.0 mm
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Other:
- net class D removed
- net class Default removed
- net class Power removed

Commit message: repositioned avr header
Parts:
- moved J2 2.98 mm to (2.54, 22.2)
Routing:
- net +5V: track 125.8 -> 129.8 mm
- net RESET: track 92.0 -> 95.3 mm
- net MOSI: track 45.5 -> 48.7 mm
- net SCK: track 46.7 -> 49.8 mm
- net MISO: track 56.3 -> 59.4 mm
- net GND: track 156.6 -> 157.7 mm
