File: pcb/bakeneko-65-pcb.kicad_sch (KiCad schematic)
At the start: 18 parts, among them J1 JST SH 4-pin, J2 AVR-ISP-6, SW1 Reset, U1 SRV05-4, U2 ATmega32U4-AU, Y1 16MHz

Commit message: pcb stuff
Parts:
- added J3: RGB Underglow, Connector_PinSocket_1.27mm:PinSocket_1x03_P1.27mm_Vertical, symbol Connector_Generic:Conn_01x03
Connections:
- net +5V: now also J3.1 (Pin_1)
- net GND: now also J3.3 (Pin_3)
- net at U2.41 (PF0): now also J3.2 (Pin_2)
- no-connect marks 4 -> 3
Changed lines of the file:
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@@
   (junction (at 58.42 81.28) (diameter 0.9144) (color 0 0 0 0)
   )
-  (no_connect (at 73.66 151.13))
   (no_connect (at 119.38 41.91))
   (no_connect (at 43.18 105.41))
@@
     (stroke (width 0) (type solid) (color 0 0 0 0))
   )
+  (wire (pts (xy 96.266 152.146) (xy 73.66 152.146))
+    (stroke (width 0) (type default) (color 0 0 0 0))
+  )
   (wire (pts (xy 31.75 115.57) (xy 43.18 115.57))
     (stroke (width 0) (type solid) (color 0 0 0 0))
@@
   (wire (pts (xy 76.2 102.87) (xy 73.66 102.87))
     (stroke (width 0) (type solid) (color 0 0 0 0))
+  )
+  (wire (pts (xy 73.66 152.146) (xy 73.66 151.13))
+    (stroke (width 0) (type default) (color 0 0 0 0))
   )
   (wire (pts (xy 76.2 153.67) (xy 73.66 153.67))
@@
     (pin "1")
   )
+  (symbol (lib_id "Connector_Generic:Conn_01x03") (at 101.346 152.146 0) (unit 1)
+    (in_bom yes) (on_board yes) (fields_autoplaced)
+    (property "Reference" "J3" (id 0) (at 103.378 151.2375 0)
+      (effects (font (size 1.27 1.27)) (justify left))
+    )
+    (property "Value" "RGB Underglow" (id 1) (at 103.378 154.0126 0)
+      (effects (font (size 1.27 1.27)) (justify left))
+    )
+    (property "Footprint" "Connector_PinSocket_1.27mm:PinSocket_1x03_P1.27mm_Vertical" (id 2) (at 101.346 152.146 0)
+      (effects (font (size 1.27 1.27)) hide)
+    )
+    (property "Datasheet" "~" (id 3) (at 101.346 152.146 0)
+      (effects (font (size 1.27 1.27)) hide)
+    )
+    (pin "1")
+    (pin "2")
+    (pin "3")
+  )
+  (symbol (lib_id "power:GND") (at 96.266 154.686 270) (unit 1)
+    (in_bom yes) (on_board yes)
+    (property "Reference" "#PWR0108" (id 0) (at 89.916 154.686 0)
+      (effects (font (size 1.27 1.27)) hide)
+    )
+    (property "Value" "GND" (id 1) (at 93.0148 154.813 0))
+    (property "Footprint" "" (id 2) (at 96.266 154.686 0)
+      (effects (font (size 1.27 1.27)) hide)
+    )
+    (property "Datasheet" "" (id 3) (at 96.266 154.686 0)
+      (effects (font (size 1.27 1.27)) hide)
+    )
+    (pin "1")
+  )
+  (symbol (lib_id "power:+5V") (at 96.266 149.606 90) (unit 1)
+    (in_bom yes) (on_board yes)
+    (property "Reference" "#PWR0109" (id 0) (at 100.076 149.606 0)
+      (effects (font (size 1.27 1.27)) hide)
+    )
+    (property "Value" "+5V" (id 1) (at 91.8718 149.225 0))
+    (property "Footprint" "" (id 2) (at 96.266 149.606 0)
+      (effects (font (size 1.27 1.27)) hide)
+    )
+    (property "Datasheet" "" (id 3) (at 96.266 149.606 0)
+      (effects (font (size 1.27 1.27)) hide)
+    )
+    (pin "1")
+  )
   (sheet (at 185.42 87.63) (size 45.72 53.34)
     (stroke (width 0) (type solid) (color 0 0 0 0))
@@
       (reference "#PWR0107") (unit 1) (value "+5V") (footprint "")
     )
+    (path "/31211d24-0284-43fc-85f9-0dda37b5537c"
+      (reference "#PWR0108") (unit 1) (value "GND") (footprint "")
+    )
+    (path "/c6e080f2-c535-4467-98bf-40ee712b30f3"
+      (reference "#PWR0109") (unit 1) (value "+5V") (footprint "")
+    )
     (path "/00000000-0000-0000-0000-00005f24d3a7"
       (reference "C1") (unit 1) (value "0.1u") (footprint "Capacitor_SMD:C_0805_2012Metric")
@@
       (reference "J2") (unit 1) (value "AVR-ISP-6") (footprint "bakeneko:ISP")
     )
+    (path "/16feeb4f-2431-4af7-a0bb-cc04a15125b5"
+      (reference "J3") (unit 1) (value "RGB Underglow") (footprint "Connector_PinSocket_1.27mm:PinSocket_1x03_P1.27mm_Vertical")
+    )
     (path "/00000000-0000-0000-0000-00005f45b9b8/00000000-0000-0000-0000-00005f497539"
